File: KiCad/ArxKey.kicad_pcb (KiCad board)
At the start: 2 copper layers, 123 parts, among them SW1 SW_Push, SW10 SW_Push, SW11 SW_Push, SW12 SW_Push, SW13 SW_Push, SW14 SW_Push, SW15 SW_Push, SW16 SW_Push, SW17 SW_Push, SW18 SW_Push, SW19 SW_Push, SW2 SW_Push, SW20 SW_Push, SW21 SW_Push, SW22 SW_Push, SW23 SW_Push, SW24 SW_Push, SW25 SW_Push, SW26 SW_Push, SW27 SW_Push, SW28 SW_Push, SW29 SW_Push, SW3 SW_Push, SW30 SW_Push, SW31 SW_Push, SW32 SW_Push, SW33 SW_Push, SW34 SW_Push, SW35 SW_Push, SW36 SW_Push, SW37 SW_Push, SW38 SW_Push, SW39 SW_Push, SW4 SW_Push, SW40 SW_Push, SW41 SW_Push, SW42 SW_Push, SW43 SW_Push, SW44 SW_Push, SW45 SW_Push, SW46 SW_Push, SW47 SW_Push, SW48 SW_Push, SW49 SW_Push, SW5 SW_Push, SW50 SW_Push, SW51 SW_Push, SW52 SW_Push, SW6 SW_Push, SW7 SW_Push, SW8 SW_Push, SW9 SW_Push, U1 XIAO-nRF52840-SMD, U2 XIAO-nRF52840-SMD

Commit message: PCB Updates
Parts:
- removed BO1, BO2, BO3: break off, Panelization.pretty-master:mouse-bite-5mm-slot
- removed H10, H8, H9: MountingHole, MountingHole:MountingHole_3.2mm_M3
- added D53: D, Diode_SMD:D_SOD-123, B.Cu at (156.1, 158.1)
- added D54: D, Diode_SMD:D_SOD-123, B.Cu at (235.7, 159.7)
- added SW53: SW_Push, PCM_marbastlib-mx:SW_MX_HS_KS-2P02B01-01_1u, F.Cu at (165.7, 158.8)
- added SW54: SW_Push, PCM_marbastlib-mx:SW_MX_HS_KS-2P02B01-01_1u, F.Cu at (225.6, 158.2)
- D1, D10, D11, D12, D13, D14, D15, D16, D17, D18, D19, D2, D20, D21, D22, D23, D24, D25, D26, D27, D28, D29, D3, D30, D31, D32, D33, D34, D35, D36, D37, D38, D39, D4, D40, D41, D42, D43, D44, D45, D46, D47, D48, D49, D5, D50, D51, D52, D6, D7, D8, D9: moved to B.Cu
- H5, H6, H7: footprint MountingHole:MountingHole_3.2mm_M3 -> Panelization.pretty-master:mouse-bite-2mm-slot
- moved SW51 264.7 mm to (244.6, 153.4), turned to 10 degrees
- moved SW11 261.9 mm to (247.0, 74.8)
- moved SW23 261.9 mm to (247.0, 93.9)
- moved SW35 261.9 mm to (247.0, 112.9)
- moved SW47 261.9 mm to (247.0, 132.0)
- moved SW22 224.9 mm to (266.1, 89.1)
- moved SW34 224.9 mm to (266.1, 108.2)
- moved SW46 224.9 mm to (266.1, 127.2)
- moved SW8 224.9 mm to (266.1, 70.0)
- moved SW21 188.3 mm to (285.1, 93.5), turned to 0 degrees
- moved SW33 188.3 mm to (285.1, 112.6)
- moved SW45 188.3 mm to (285.1, 131.6)
- moved SW7 188.3 mm to (285.1, 74.5)
- moved SW20 152.5 mm to (304.2, 98.9)
- moved SW32 152.5 mm to (304.2, 118.0)
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Routing:
- net /left/COL5: track 0.00 -> 275.4 mm
- net /left/COL4: track 0.00 -> 245.3 mm
- net /left/COL3: track 0.00 -> 220.7 mm
- net /right/ROW3: track 0.00 -> 210.4 mm, vias 0 -> 1
- net /right/COL4: track 0.00 -> 208.8 mm, vias 0 -> 2
- net /right/COL5: track 0.00 -> 207.1 mm, vias 0 -> 2
- net /right/COL3: track 0.00 -> 204.3 mm, vias 0 -> 2
- net /right/COL0: track 0.00 -> 193.4 mm
- net /right/ROW2: track 0.00 -> 191.9 mm, vias 0 -> 1
- net /right/COL1: track 0.00 -> 183.3 mm, vias 0 -> 2
- net /left/ROW3: track 0.00 -> 177.9 mm, vias 0 -> 1
- net /right/ROW0: track 0.00 -> 169.2 mm, vias 0 -> 1
- net /right/COL2: track 0.00 -> 167.2 mm, vias 0 -> 2
- net /left/ROW0: track 0.00 -> 164.7 mm, vias 0 -> 1
- net /left/ROW2: track 0.00 -> 163.7 mm, vias 0 -> 1
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Other:
- board outline added: 280.5 x 117 mm
