File: KiCad/ArxKey.kicad_sch (KiCad schematic)
At the start: 3 parts

Commit message: PCB Updates
Parts:
- removed BO1, BO2, BO3: break off, Panelization.pretty-master:mouse-bite-5mm-slot, symbol Mechanical:MountingHole
- added H5, H6, H7: MountingHole, Panelization.pretty-master:mouse-bite-2mm-slot, symbol Mechanical:MountingHole
Changed lines of the file:
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@@
 	(symbol
 		(lib_id "Mechanical:MountingHole")
-		(at 85.09 97.79 0)
+		(at 63.5 96.52 0)
 		(unit 1)
 		(body_style 1)
@@
 		(dnp no)
 		(fields_autoplaced yes)
-		(property "Reference" "BO2"
-			(at 87.63 96.5199 0)
-			(show_name no)
-			(do_not_autoplace no)
-			(effects
-				(font
-					(size 1.27 1.27)
-				)
-				(justify left)
-			)
-		)
-		(property "Value" "break off"
-			(at 87.63 99.0599 0)
-			(show_name no)
-			(do_not_autoplace no)
-			(effects
-				(font
-					(size 1.27 1.27)
-				)
-				(justify left)
-			)
-		)
-		(property "Footprint" "Panelization.pretty-master:mouse-bite-5mm-slot"
-			(at 85.09 97.79 0)
+		(property "Reference" "H5"
+			(at 66.04 95.2499 0)
+			(show_name no)
+			(do_not_autoplace no)
+			(effects
+				(font
+					(size 1.27 1.27)
+				)
+				(justify left)
+			)
+		)
+		(property "Value" "MountingHole"
+			(at 66.04 97.7899 0)
+			(show_name no)
+			(do_not_autoplace no)
+			(effects
+				(font
+					(size 1.27 1.27)
+				)
+				(justify left)
+			)
+		)
+		(property "Footprint" "Panelization.pretty-master:mouse-bite-2mm-slot"
+			(at 63.5 96.52 0)
 			(hide yes)
 			(show_name no)
@@
 		)
 		(property "Datasheet" ""
-			(at 85.09 97.79 0)
+			(at 63.5 96.52 0)
 			(hide yes)
 			(show_name no)
@@
 		)
 		(property "Description" "Mounting Hole without connection"
-			(at 85.09 97.79 0)
+			(at 63.5 96.52 0)
 			(hide yes)
 			(show_name no)
@@
 			(project "ArxKey"
 				(path "/23ad1585-5c91-4de6-86f2-a576fc0b31a5"
-					(reference "BO2")
+					(reference "H5")
 					(unit 1)
 				)
@@
 	(symbol
 		(lib_id "Mechanical:MountingHole")
-		(at 85.09 91.44 0)
+		(at 63.5 109.22 0)
 		(unit 1)
 		(body_style 1)
@@
 		(dnp no)
 		(fields_autoplaced yes)
-		(property "Reference" "BO1"
-			(at 87.63 90.1699 0)
-			(show_name no)
-			(do_not_autoplace no)
-			(effects
-				(font
-					(size 1.27 1.27)
-				)
-				(justify left)
-			)
-		)
-		(property "Value" "break off"
-			(at 87.63 92.7099 0)
-			(show_name no)
-			(do_not_autoplace no)
-			(effects
-				(font
-					(size 1.27 1.27)
-				)
-				(justify left)
-			)
-		)
-		(property "Footprint" "Panelization.pretty-master:mouse-bite-5mm-slot"
-			(at 85.09 91.44 0)
+		(property "Reference" "H7"
+			(at 66.04 107.9499 0)
+			(show_name no)
+			(do_not_autoplace no)
+			(effects
+				(font
+					(size 1.27 1.27)
+				)
+				(justify left)
+			)
+		)
+		(property "Value" "MountingHole"
+			(at 66.04 110.4899 0)
+			(show_name no)
+			(do_not_autoplace no)
+			(effects
+				(font
+					(size 1.27 1.27)
+				)
+				(justify left)
+			)
+		)
+		(property "Footprint" "Panelization.pretty-master:mouse-bite-2mm-slot"
+			(at 63.5 109.22 0)
 			(hide yes)
 			(show_name no)
@@
 		)
 		(property "Datasheet" ""
-			(at 85.09 91.44 0)
+			(at 63.5 109.22 0)
 			(hide yes)
 			(show_name no)
@@
 		)
 		(property "Description" "Mounting Hole without connection"
-			(at 85.09 91.44 0)
+			(at 63.5 109.22 0)
 			(hide yes)
 			(show_name no)
@@
 			(project "ArxKey"
 				(path "/23ad1585-5c91-4de6-86f2-a576fc0b31a5"
-					(reference "BO1")
+					(reference "H7")
 					(unit 1)
 				)
@@
 	(symbol
 		(lib_id "Mechanical:MountingHole")
-		(at 85.09 104.14 0)
+		(at 63.5 102.87 0)
 		(unit 1)
 		(body_style 1)
@@
 		(dnp no)
 		(fields_autoplaced yes)
-		(property "Reference" "BO3"
-			(at 87.63 102.8699 0)
-			(show_name no)
-			(do_not_autoplace no)
-			(effects
-				(font
-					(size 1.27 1.27)
-				)
-				(justify left)
-			)
-		)
-		(property "Value" "break off"
-			(at 87.63 105.4099 0)
-			(show_name no)
-			(do_not_autoplace no)
-			(effects
-				(font
-					(size 1.27 1.27)
-				)
-				(justify left)
-			)
-		)
-		(property "Footprint" "Panelization.pretty-master:mouse-bite-5mm-slot"
-			(at 85.09 104.14 0)
+		(property "Reference" "H6"
+			(at 66.04 101.5999 0)
+			(show_name no)
+			(do_not_autoplace no)
+			(effects
+				(font
+					(size 1.27 1.27)
+				)
+				(justify left)
+			)
+		)
+		(property "Value" "MountingHole"
+			(at 66.04 104.1399 0)
+			(show_name no)
+			(do_not_autoplace no)
+			(effects
+				(font
+					(size 1.27 1.27)
+				)
+				(justify left)
+			)
+		)
+		(property "Footprint" "Panelization.pretty-master:mouse-bite-2mm-slot"
+			(at 63.5 102.87 0)
 			(hide yes)
 			(show_name no)
@@
 		)
 		(property "Datasheet" ""
-			(at 85.09 104.14 0)
+			(at 63.5 102.87 0)
 			(hide yes)
 			(show_name no)
@@
 		)
 		(property "Description" "Mounting Hole without connection"
-			(at 85.09 104.14 0)
+			(at 63.5 102.87 0)
 			(hide yes)
 			(show_name no)
@@
 			(project "ArxKey"
 				(path "/23ad1585-5c91-4de6-86f2-a576fc0b31a5"
-					(reference "BO3")
+					(reference "H6")
 					(unit 1)
 				)
