File: KiCad/side.kicad_sch (KiCad schematic)
At the start: 60 parts, among them SW1 SW_Push, SW10 SW_Push, SW13 SW_Push, SW14 SW_Push, SW15 SW_Push, SW16 SW_Push, SW17 SW_Push, SW18 SW_Push, SW25 SW_Push, SW26 SW_Push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

Commit message: PCB Updates
Parts:
- removed H5, H6, H9: MountingHole, MountingHole:MountingHole_3.2mm_M3, symbol Mechanical:MountingHole
- added D53: D, Diode_SMD:D_SOD-123, symbol Device:D
- added SW53: SW_Push, PCM_marbastlib-mx:SW_MX_HS_KS-2P02B01-01_1u, symbol Switch:SW_Push
Connections:
- net COL3: now also SW53.1
- net ROW4: now also D53.1 (K)
- new net: D53.2 (A), SW53.2
